Commit message: Finished

File: body.urdf (robot description, URDF)
Before this commit: robot robot, 9 links, 8 joints
Links:
- added link Link9, mass 1; collision box size=0.9992792389069787 0.6857346745655395 0.5799256477059034; visual box size=0.9992792389069787 0.6857346745655395 0.5799256477059034
- link Link0: geometry collision box size=0.6417011747789898 0.7612488328243612 0.4170170537184503; visual box size=0.6417011747789898 0.7612488328243612 0.4170170537184503
- link Link1: geometry collision box size=0.6417011747789898 0.7612488328243612 0.4170170537184503; visual box size=0.6417011747789898 0.7612488328243612 0.4170170537184503
- link Link2: geometry collision box size=0.5765343361739661 0.38569008827215906 0.40920614486075374; visual box size=0.5765343361739661 0.38569008827215906 0.40920614486075374
- link Link3: geometry collision box size=0.7754177525054313 0.6589628071244793 0.7976606941190332; visual box size=0.7754177525054313 0.6589628071244793 0.7976606941190332
- link Link4: geometry collision box size=0.27802072478833184 0.6165260371228417 0.5956028716734549; visual box size=0.27802072478833184 0.6165260371228417 0.5956028716734549
- link Link5: geometry collision box size=0.8658515673682667 0.4476108490243612 0.8370084584328239; visual box size=0.8658515673682667 0.4476108490243612 0.8370084584328239
- link Link6: geometry collision box size=0.36996110147554084 0.6808333274219343 0.9787625660494244; visual box size=0.36996110147554084 0.6808333274219343 0.9787625660494244
- link Link7: geometry collision box size=0.8262967813995687 0.5395425079297842 0.8608864424021148; visual box size=0.8262967813995687 0.5395425079297842 0.8608864424021148
- link Link8: geometry collision box size=0.55746998417317 0.8718372186383003 0.20180988775649755; visual box size=0.55746998417317 0.8718372186383003 0.20180988775649755
Joints:
- added joint Link8_Link9: type revolute, parent Link8, child Link9, origin xyz=-0.278734992086585 -0.43591860931915016 0.0 rpy=0 0 0, axis 0 1 0, limit lower=-3.14159 upper=3.14159 effort=0.0 velocity=0.0
- joint Link0_Link1: origin xyz=-0.5932757055308087 0 0.17983265740333676 rpy=0 0 0 -> xyz=0.3208505873894949 0 1.4170170537184503 rpy=0 0 0
- joint Link1_Link2: origin xyz=-0.38545724381974966 0 0.1207142322209791 rpy=0 0 0 -> xyz=0.3208505873894949 0.3806244164121806 0.0 rpy=0 0 0
- joint Link2_Link3: origin xyz=-0.9006586223149269 0 0.04444577146793727 rpy=0 0 0 -> xyz=-0.28826716808698305 0.19284504413607953 0.40920614486075374 rpy=0 0 0
- joint Link3_Link4: origin xyz=-0.8815050146407164 0 -0.007945603082792907 rpy=0 0 0 -> xyz=-0.7754177525054313 0 0.0 rpy=0 0 0
- joint Link4_Link5: origin xyz=-0.3940096721560262 0 -0.05950821081159513 rpy=0 0 0 -> xyz=0.0 0 0.5956028716734549 rpy=0 0 0
- joint Link5_Link6: origin xyz=-0.832446402406767 0 -0.16734604185324858 rpy=0 0 0 -> xyz=0.43292578368413337 0.2238054245121806 0.8370084584328239 rpy=0 0 0
- joint Link6_Link7: origin xyz=-0.36030463637147503 0 0.1406954023945549 rpy=0 0 0 -> xyz=0 0.0 0.9787625660494244 rpy=0 0 0
- joint Link7_Link8: origin xyz=-0.8909637190300066 0 0.23058638896260564 rpy=0 0 0 -> xyz=-0.4131483906997844 -0.2697712539648921 0.0 rpy=0 0 0

Commit message: Collision check

File: body.urdf (robot description, URDF)
Before this commit: robot robot, 10 links, 9 joints
Links:
- added link Link10, mass 1; collision box size=0.6625012369906736 0.5746050280471076 0.45580482206979345; visual box size=0.6625012369906736 0.5746050280471076 0.45580482206979345
- added link Link11, mass 1; collision box size=0.5822929722547812 0.4269349545750995 0.4851502454877474; visual box size=0.5822929722547812 0.4269349545750995 0.4851502454877474
- added link Link12, mass 1; collision box size=0.47541097157136747 0.7844274977050039 0.52508077185515; visual box size=0.47541097157136747 0.7844274977050039 0.52508077185515
- added link Link13, mass 1; collision box size=0.45500477009937157 0.3400579960825105 0.5566165245961499; visual box size=0.45500477009937157 0.3400579960825105 0.5566165245961499
- added link Link14, mass 1; collision box size=0.6857752063318754 0.47076037115527947 0.8624473333741574; visual box size=0.6857752063318754 0.47076037115527947 0.8624473333741574
- added link Link15, mass 1; collision box size=0.41074331599299657 0.27055787298093875 0.4848058256907374; visual box size=0.41074331599299657 0.27055787298093875 0.4848058256907374
- added link Link16, mass 1; collision box size=0.33589292926711045 0.5051427833419606 0.40341121990226636; visual box size=0.33589292926711045 0.5051427833419606 0.40341121990226636
- added link Link17, mass 1; collision box size=0.4239106972274379 0.3031061575525593 0.5294503713545683; visual box size=0.4239106972274379 0.3031061575525593 0.5294503713545683
- link Link0: geometry collision box size=0.9376410895639657 0.26117246902533187 0.8969598027004575; visual box size=0.9376410895639657 0.26117246902533187 0.8969598027004575
- link Link1: geometry collision box size=0.9376410895639657 0.26117246902533187 0.8969598027004575; visual box size=0.9376410895639657 0.26117246902533187 0.8969598027004575
- link Link2: geometry collision box size=0.26784671081220623 0.3530119165640366 0.5171965147517983; visual box size=0.26784671081220623 0.3530119165640366 0.5171965147517983
- link Link3: geometry collision box size=0.684937839215916 0.5959936872934106 0.5917814332374245; visual box size=0.684937839215916 0.5959936872934106 0.5917814332374245
- link Link4: geometry collision box size=0.21174473302095703 0.3817530001388617 0.9767779485604131; visual box size=0.21174473302095703 0.3817530001388617 0.9767779485604131
- link Link5: geometry collision box size=0.6938926207922318 0.4898461664274096 0.657987726445438; visual box size=0.6938926207922318 0.4898461664274096 0.657987726445438
- link Link6: geometry collision box size=0.7309508200198964 0.2937315683503974 0.4248533043200622; visual box size=0.7309508200198964 0.2937315683503974 0.4248533043200622
- link Link7: geometry collision box size=0.6474227125826808 0.4920934200385169 0.6861072290027983; visual box size=0.6474227125826808 0.4920934200385169 0.6861072290027983
- link Link8: geometry collision box size=0.7360566883716031 0.4160761015502818 0.44750976721783353; visual box size=0.7360566883716031 0.4160761015502818 0.44750976721783353
- link Link9: geometry collision box size=0.7689076917583233 0.2778093854430075 0.5418321264658441; visual box size=0.7689076917583233 0.2778093854430075 0.5418321264658441
Joints:
- added joint Link10_Link11: type revolute, parent Link10, child Link11, origin xyz=0.3312506184953368 0.2873025140235538 0.0 rpy=0 0 0, axis 0 1 0, limit lower=-3.14159 upper=3.14159 effort=0.0 velocity=0.0
- added joint Link11_Link12: type revolute, parent Link11, child Link12, origin xyz=0.0 0 0.0 rpy=0 0 0, axis 0 1 0, limit lower=-3.14159 upper=3.14159 effort=0.0 velocity=0.0
- added joint Link12_Link13: type revolute, parent Link12, child Link13, origin xyz=0.0 0 0.0 rpy=0 0 0, axis 0 1 0, limit lower=-3.14159 upper=3.14159 effort=0.0 velocity=0.0
- added joint Link13_Link14: type revolute, parent Link13, child Link14, origin xyz=0.45500477009937157 0 0.0 rpy=0 0 0, axis 0 1 0, limit lower=-3.14159 upper=3.14159 effort=0.0 velocity=0.0
- added joint Link14_Link15: type revolute, parent Link14, child Link15, origin xyz=0.0 0 0.8624473333741574 rpy=0 0 0, axis 0 1 0, limit lower=-3.14159 upper=3.14159 effort=0.0 velocity=0.0
- added joint Link15_Link16: type revolute, parent Link15, child Link16, origin xyz=-0.20537165799649829 -0.13527893649046938 0.4848058256907374 rpy=0 0 0, axis 0 1 0, limit lower=-3.14159 upper=3.14159 effort=0.0 velocity=0.0
- added joint Link16_Link17: type revolute, parent Link16, child Link17, origin xyz=0 -0.5051427833419606 0.0 rpy=0 0 0, axis 0 1 0, limit lower=-3.14159 upper=3.14159 effort=0.0 velocity=0.0
- added joint Link9_Link10: type revolute, parent Link9, child Link10, origin xyz=0.38445384587916165 0.13890469272150374 0.0 rpy=0 0 0, axis 0 1 0, limit lower=-3.14159 upper=3.14159 effort=0.0 velocity=0.0
- joint Link0_Link1: origin xyz=0.3208505873894949 0 1.4170170537184503 rpy=0 0 0 -> xyz=0.4688205447819829 0 1.8969598027004575 rpy=0 0 0
- joint Link1_Link2: origin xyz=0.3208505873894949 0.3806244164121806 0.0 rpy=0 0 0 -> xyz=0.0 0 0.0 rpy=0 0 0
- joint Link2_Link3: origin xyz=-0.28826716808698305 0.19284504413607953 0.40920614486075374 rpy=0 0 0 -> xyz=-0.13392335540610312 0.1765059582820183 0.5171965147517983 rpy=0 0 0
- joint Link3_Link4: origin xyz=-0.7754177525054313 0 0.0 rpy=0 0 0 -> xyz=0 0.0 0.5917814332374245 rpy=0 0 0
- joint Link4_Link5: origin xyz=0.0 0 0.5956028716734549 rpy=0 0 0 -> xyz=0 -0.3817530001388617 0.9767779485604131 rpy=0 0 0
- joint Link5_Link6: origin xyz=0.43292578368413337 0.2238054245121806 0.8370084584328239 rpy=0 0 0 -> xyz=0.3469463103961159 -0.2449230832137048 0.657987726445438 rpy=0 0 0
- joint Link6_Link7: origin xyz=0 0.0 0.9787625660494244 rpy=0 0 0 -> xyz=0.7309508200198964 0 0.0 rpy=0 0 0
- joint Link7_Link8: origin xyz=-0.4131483906997844 -0.2697712539648921 0.0 rpy=0 0 0 -> xyz=0.3237113562913404 -0.24604671001925846 0.6861072290027983 rpy=0 0 0
- joint Link8_Link9: origin xyz=-0.278734992086585 -0.43591860931915016 0.0 rpy=0 0 0 -> xyz=0.36802834418580155 -0.2080380507751409 0.0 rpy=0 0 0

Commit message: Added readme

File: body.urdf (robot description, URDF)
Before this commit: robot robot, 18 links, 17 joints
Links:
- removed link Link10
- removed link Link11
- removed link Link12
- removed link Link13
- removed link Link14
- removed link Link15
- removed link Link16
- removed link Link17
- removed link Link7
- removed link Link8
- removed link Link9
- link Link0: geometry collision box size=0.9208522992814163 0.842108870625714 0.6969090363245609; visual box size=0.9208522992814163 0.842108870625714 0.6969090363245609
- link Link1: geometry collision box size=0.9208522992814163 0.842108870625714 0.6969090363245609; visual box size=0.9208522992814163 0.842108870625714 0.6969090363245609
- link Link2: geometry collision box size=0.8555121533969403 0.2478687622635196 0.588479008670083; visual box size=0.8555121533969403 0.2478687622635196 0.588479008670083
- link Link3: geometry collision box size=0.6991089078896957 0.3088754723382045 0.8616077939475684; visual box size=0.6991089078896957 0.3088754723382045 0.8616077939475684
- link Link4: geometry collision box size=0.6421979722854341 0.9209424257362144 0.4773653620351923; visual box size=0.6421979722854341 0.9209424257362144 0.4773653620351923
- link Link5: geometry collision box size=0.3266180409586175 0.93281366886578 0.8918690049363385; visual box size=0.3266180409586175 0.93281366886578 0.8918690049363385
- link Link6: geometry collision box size=0.37254078302395927 0.20206073729232232 0.8153665748501777; visual box size=0.37254078302395927 0.20206073729232232 0.8153665748501777
Joints:
- removed joint Link10_Link11
- removed joint Link11_Link12
- removed joint Link12_Link13
- removed joint Link13_Link14
- removed joint Link14_Link15
- removed joint Link15_Link16
- removed joint Link16_Link17
- removed joint Link6_Link7
- removed joint Link7_Link8
- removed joint Link8_Link9
- removed joint Link9_Link10
- joint Link0_Link1: origin xyz=0.4688205447819829 0 1.8969598027004575 rpy=0 0 0 -> xyz=0.46042614964070816 0 1.696909036324561 rpy=0 0 0
- joint Link1_Link2: origin xyz=0.0 0 0.0 rpy=0 0 0 -> xyz=0.9208522992814163 0 0.0 rpy=0 0 0
- joint Link2_Link3: origin xyz=-0.13392335540610312 0.1765059582820183 0.5171965147517983 rpy=0 0 0 -> xyz=0.8555121533969403 0 0.0 rpy=0 0 0
- joint Link3_Link4: origin xyz=0 0.0 0.5917814332374245 rpy=0 0 0 -> xyz=0.34955445394484785 0.15443773616910225 0.8616077939475684 rpy=0 0 0
- joint Link4_Link5: origin xyz=0 -0.3817530001388617 0.9767779485604131 rpy=0 0 0 -> xyz=0.32109898614271704 0.4604712128681072 0.0 rpy=0 0 0
- joint Link5_Link6: origin xyz=0.3469463103961159 -0.2449230832137048 0.657987726445438 rpy=0 0 0 -> xyz=0.16330902047930876 -0.46640683443289 0.0 rpy=0 0 0

Commit message: Checkpoint

File: body.urdf (robot description, URDF)
Before this commit: robot robot, 7 links, 6 joints
Links:
- removed link Link2
- removed link Link3
- removed link Link4
- removed link Link5
- removed link Link6
- link Link0: geometry collision box size=0.26930194887184805 1.5951329881470557 0.49164627665217076; visual box size=0.26930194887184805 1.5951329881470557 0.49164627665217076
- link Link1: geometry collision box size=1.545246488338602 0.8379783736586159 1.094826110632794; visual box size=1.545246488338602 0.8379783736586159 1.094826110632794
Joints:
- removed joint Link1_Link2
- removed joint Link2_Link3
- removed joint Link3_Link4
- removed joint Link4_Link5
- removed joint Link5_Link6
- joint Link0_Link1: origin xyz=0.46042614964070816 0 1.696909036324561 rpy=0 0 0 -> xyz=0.13465097443592403 0 0.547413055316397 rpy=0 0 0
