Commit message: Done

File: body.urdf (robot description, URDF)
Before this commit: robot robot, 2 links, 1 joints
Links:
- added link Link1TwoLink0, mass 1; collision box size=1.115133581989522 0.6926171844667286 0.6179836134638079; visual box size=1.115133581989522 0.6926171844667286 0.6179836134638079
- added link Link1TwoLink1, mass 1; collision box size=1.115133581989522 0.6926171844667286 0.6179836134638079; visual box size=1.115133581989522 0.6926171844667286 0.6179836134638079
- added link Link1TwoLink2, mass 1; collision box size=1.115133581989522 0.6926171844667286 0.6179836134638079; visual box size=1.115133581989522 0.6926171844667286 0.6179836134638079
- added link Link1TwoLink3, mass 1; collision box size=1.115133581989522 0.6926171844667286 0.6179836134638079; visual box size=1.115133581989522 0.6926171844667286 0.6179836134638079
- added link Link1TwoLink4, mass 1; collision box size=1.115133581989522 0.6926171844667286 0.6179836134638079; visual box size=1.115133581989522 0.6926171844667286 0.6179836134638079
- added link Link1ZeroLink0, mass 1; collision box size=0.6245578238503056 0.8309183632281945 0.5587460820760188; visual box size=0.6245578238503056 0.8309183632281945 0.5587460820760188
- added link Link2, mass 1; collision box size=1.2987328958406814 1.4283480197268903 0.9881684406294893; visual box size=1.2987328958406814 1.4283480197268903 0.9881684406294893
- added link Link2TwoLink0, mass 1; collision box size=1.1024409726377706 0.33794875175027567 0.7326903474578026; visual box size=1.1024409726377706 0.33794875175027567 0.7326903474578026
- added link Link2TwoLink1, mass 1; collision box size=1.1024409726377706 0.33794875175027567 0.7326903474578026; visual box size=1.1024409726377706 0.33794875175027567 0.7326903474578026
- added link Link2TwoLink2, mass 1; collision box size=1.1024409726377706 0.33794875175027567 0.7326903474578026; visual box size=1.1024409726377706 0.33794875175027567 0.7326903474578026
- added link Link2ZeroLink0, mass 1; collision box size=0.7909559601568661 0.4588162710567005 0.22808589092273684; visual box size=0.7909559601568661 0.4588162710567005 0.22808589092273684
- added link Link3, mass 1; collision box size=1.569495597626496 1.4578655587551734 0.43501387901448185; visual box size=1.569495597626496 1.4578655587551734 0.43501387901448185
- added link Link3OneLink0, mass 1; collision box size=0.893186047551715 0.4047008304167928 1.0947954316146549; visual box size=0.893186047551715 0.4047008304167928 1.0947954316146549
- added link Link3TwoLink0, mass 1; collision box size=0.4924400623740139 0.39198652225098635 0.8844546984555164; visual box size=0.4924400623740139 0.39198652225098635 0.8844546984555164
- added link Link3TwoLink1, mass 1; collision box size=0.4924400623740139 0.39198652225098635 0.8844546984555164; visual box size=0.4924400623740139 0.39198652225098635 0.8844546984555164
- added link Link3TwoLink2, mass 1; collision box size=0.4924400623740139 0.39198652225098635 0.8844546984555164; visual box size=0.4924400623740139 0.39198652225098635 0.8844546984555164
- added link Link3TwoLink3, mass 1; collision box size=0.4924400623740139 0.39198652225098635 0.8844546984555164; visual box size=0.4924400623740139 0.39198652225098635 0.8844546984555164
- added link Link3TwoLink4, mass 1; collision box size=0.4924400623740139 0.39198652225098635 0.8844546984555164; visual box size=0.4924400623740139 0.39198652225098635 0.8844546984555164
- added link Link3ZeroLink0, mass 1; collision box size=0.5193562998568066 0.5190494727808921 0.41091471067501834; visual box size=0.5193562998568066 0.5190494727808921 0.41091471067501834
- added link Link4, mass 1; collision box size=1.2084464218745348 1.2390595539877647 1.6156204905666065; visual box size=1.2084464218745348 1.2390595539877647 1.6156204905666065
- added link Link4OneLink0, mass 1; collision box size=1.1530996768260393 0.29112215744207376 0.5886243969431917; visual box size=1.1530996768260393 0.29112215744207376 0.5886243969431917
- added link Link4TwoLink0, mass 1; collision box size=0.35051662062359584 1.1177530052663003 0.45229710655044925; visual box size=0.35051662062359584 1.1177530052663003 0.45229710655044925
- added link Link4TwoLink1, mass 1; collision box size=0.35051662062359584 1.1177530052663003 0.45229710655044925; visual box size=0.35051662062359584 1.1177530052663003 0.45229710655044925
- added link Link4TwoLink2, mass 1; collision box size=0.35051662062359584 1.1177530052663003 0.45229710655044925; visual box size=0.35051662062359584 1.1177530052663003 0.45229710655044925
- added link Link4TwoLink3, mass 1; collision box size=0.35051662062359584 1.1177530052663003 0.45229710655044925; visual box size=0.35051662062359584 1.1177530052663003 0.45229710655044925
- added link Link4TwoLink4, mass 1; collision box size=0.35051662062359584 1.1177530052663003 0.45229710655044925; visual box size=0.35051662062359584 1.1177530052663003 0.45229710655044925
- added link Link4ZeroLink0, mass 1; collision box size=0.4510648672129561 0.8435444100905927 0.355915202183755; visual box size=0.4510648672129561 0.8435444100905927 0.355915202183755
- added link Link5, mass 1; collision box size=0.715790879794572 1.1210281002743023 1.5829486965180457; visual box size=0.715790879794572 1.1210281002743023 1.5829486965180457
- added link Link5TwoLink0, mass 1; collision box size=0.7438925640413505 0.7916370149226362 1.1331223389185459; visual box size=0.7438925640413505 0.7916370149226362 1.1331223389185459
- added link Link5TwoLink1, mass 1; collision box size=0.7438925640413505 0.7916370149226362 1.1331223389185459; visual box size=0.7438925640413505 0.7916370149226362 1.1331223389185459
- added link Link5TwoLink2, mass 1; collision box size=0.7438925640413505 0.7916370149226362 1.1331223389185459; visual box size=0.7438925640413505 0.7916370149226362 1.1331223389185459
- added link Link5TwoLink3, mass 1; collision box size=0.7438925640413505 0.7916370149226362 1.1331223389185459; visual box size=0.7438925640413505 0.7916370149226362 1.1331223389185459
- added link Link5TwoLink4, mass 1; collision box size=0.7438925640413505 0.7916370149226362 1.1331223389185459; visual box size=0.7438925640413505 0.7916370149226362 1.1331223389185459
- link Link0: geometry collision box size=0.34512603466571967 0.6653327633834607 1.7991030490333804; visual box size=0.34512603466571967 0.6653327633834607 1.7991030490333804
- link Link1: geometry collision box size=0.5535255234622825 1.1339874684731799 0.5970428511087296; visual box size=0.5535255234622825 1.1339874684731799 0.5970428511087296
Joints:
- added joint Link1TwoLink0_Link1TwoLink1: type revolute, parent Link1TwoLink0, child Link1TwoLink1, origin xyz=0 0 0.6179836134638079 rpy=0 0 0, axis 0 1 0, limit lower=-3.14159 upper=3.14159 effort=0.0 velocity=0.0
- added joint Link1TwoLink1_Link1TwoLink2: type revolute, parent Link1TwoLink1, child Link1TwoLink2, origin xyz=0 0 0.6179836134638079 rpy=0 0 0, axis 0 1 0, limit lower=-3.14159 upper=3.14159 effort=0.0 velocity=0.0
- added joint Link1TwoLink2_Link1TwoLink3: type revolute, parent Link1TwoLink2, child Link1TwoLink3, origin xyz=0 0 0.6179836134638079 rpy=0 0 0, axis 0 1 0, limit lower=-3.14159 upper=3.14159 effort=0.0 velocity=0.0
- added joint Link1TwoLink3_Link1TwoLink4: type revolute, parent Link1TwoLink3, child Link1TwoLink4, origin xyz=0 0 0.6179836134638079 rpy=0 0 0, axis 0 1 0, limit lower=-3.14159 upper=3.14159 effort=0.0 velocity=0.0
- added joint Link1_Link1TwoLink0: type revolute, parent Link1, child Link1TwoLink0, origin xyz=0 0.5669937342365899 0.2985214255543648 rpy=0 0 0, axis 0 1 0, limit lower=-3.14159 upper=3.14159 effort=0.0 velocity=0.0
- added joint Link1_Link1ZeroLink0: type revolute, parent Link1, child Link1ZeroLink0, origin xyz=0.2767627617311412 0.5669937342365899 0 rpy=0 0 0, axis 0 1 0, limit lower=-3.14159 upper=3.14159 effort=0.0 velocity=0.0
- added joint Link1_Link2: type revolute, parent Link1, child Link2, origin xyz=0 1.1339874684731799 0 rpy=0 0 0, axis 0 1 0, limit lower=-3.14159 upper=3.14159 effort=0.0 velocity=0.0
- added joint Link2TwoLink0_Link2TwoLink1: type revolute, parent Link2TwoLink0, child Link2TwoLink1, origin xyz=0 0 0.7326903474578026 rpy=0 0 0, axis 0 1 0, limit lower=-3.14159 upper=3.14159 effort=0.0 velocity=0.0
- added joint Link2TwoLink1_Link2TwoLink2: type revolute, parent Link2TwoLink1, child Link2TwoLink2, origin xyz=0 0 0.7326903474578026 rpy=0 0 0, axis 0 1 0, limit lower=-3.14159 upper=3.14159 effort=0.0 velocity=0.0
- added joint Link2_Link2TwoLink0: type revolute, parent Link2, child Link2TwoLink0, origin xyz=0 0.7141740098634451 0.49408422031474464 rpy=0 0 0, axis 0 1 0, limit lower=-3.14159 upper=3.14159 effort=0.0 velocity=0.0
- added joint Link2_Link2ZeroLink0: type revolute, parent Link2, child Link2ZeroLink0, origin xyz=0.6493664479203407 0.7141740098634451 0 rpy=0 0 0, axis 0 1 0, limit lower=-3.14159 upper=3.14159 effort=0.0 velocity=0.0
- added joint Link2_Link3: type revolute, parent Link2, child Link3, origin xyz=0 1.4283480197268903 0 rpy=0 0 0, axis 0 1 0, limit lower=-3.14159 upper=3.14159 effort=0.0 velocity=0.0
- added joint Link3TwoLink0_Link3TwoLink1: type revolute, parent Link3TwoLink0, child Link3TwoLink1, origin xyz=0 0 0.8844546984555164 rpy=0 0 0, axis 0 1 0, limit lower=-3.14159 upper=3.14159 effort=0.0 velocity=0.0
- added joint Link3TwoLink1_Link3TwoLink2: type revolute, parent Link3TwoLink1, child Link3TwoLink2, origin xyz=0 0 0.8844546984555164 rpy=0 0 0, axis 0 1 0, limit lower=-3.14159 upper=3.14159 effort=0.0 velocity=0.0
- added joint Link3TwoLink2_Link3TwoLink3: type revolute, parent Link3TwoLink2, child Link3TwoLink3, origin xyz=0 0 0.8844546984555164 rpy=0 0 0, axis 0 1 0, limit lower=-3.14159 upper=3.14159 effort=0.0 velocity=0.0
- added joint Link3TwoLink3_Link3TwoLink4: type revolute, parent Link3TwoLink3, child Link3TwoLink4, origin xyz=0 0 0.8844546984555164 rpy=0 0 0, axis 0 1 0, limit lower=-3.14159 upper=3.14159 effort=0.0 velocity=0.0
- added joint Link3_Link3OneLink0: type revolute, parent Link3, child Link3OneLink0, origin xyz=-0.784747798813248 0.7289327793775867 0 rpy=0 0 0, axis 0 1 0, limit lower=-3.14159 upper=3.14159 effort=0.0 velocity=0.0
- added joint Link3_Link3TwoLink0: type revolute, parent Link3, child Link3TwoLink0, origin xyz=0 0.7289327793775867 0.21750693950724093 rpy=0 0 0, axis 0 1 0, limit lower=-3.14159 upper=3.14159 effort=0.0 velocity=0.0
- added joint Link3_Link3ZeroLink0: type revolute, parent Link3, child Link3ZeroLink0, origin xyz=0.784747798813248 0.7289327793775867 0 rpy=0 0 0, axis 0 1 0, limit lower=-3.14159 upper=3.14159 effort=0.0 velocity=0.0
- added joint Link3_Link4: type revolute, parent Link3, child Link4, origin xyz=0 1.4578655587551734 0 rpy=0 0 0, axis 0 1 0, limit lower=-3.14159 upper=3.14159 effort=0.0 velocity=0.0
- added joint Link4TwoLink0_Link4TwoLink1: type revolute, parent Link4TwoLink0, child Link4TwoLink1, origin xyz=0 0 0.45229710655044925 rpy=0 0 0, axis 0 1 0, limit lower=-3.14159 upper=3.14159 effort=0.0 velocity=0.0
- added joint Link4TwoLink1_Link4TwoLink2: type revolute, parent Link4TwoLink1, child Link4TwoLink2, origin xyz=0 0 0.45229710655044925 rpy=0 0 0, axis 0 1 0, limit lower=-3.14159 upper=3.14159 effort=0.0 velocity=0.0
- added joint Link4TwoLink2_Link4TwoLink3: type revolute, parent Link4TwoLink2, child Link4TwoLink3, origin xyz=0 0 0.45229710655044925 rpy=0 0 0, axis 0 1 0, limit lower=-3.14159 upper=3.14159 effort=0.0 velocity=0.0
- added joint Link4TwoLink3_Link4TwoLink4: type revolute, parent Link4TwoLink3, child Link4TwoLink4, origin xyz=0 0 0.45229710655044925 rpy=0 0 0, axis 0 1 0, limit lower=-3.14159 upper=3.14159 effort=0.0 velocity=0.0
- added joint Link4_Link4OneLink0: type revolute, parent Link4, child Link4OneLink0, origin xyz=-0.6042232109372674 0.6195297769938823 0 rpy=0 0 0, axis 0 1 0, limit lower=-3.14159 upper=3.14159 effort=0.0 velocity=0.0
- added joint Link4_Link4TwoLink0: type revolute, parent Link4, child Link4TwoLink0, origin xyz=0 0.6195297769938823 0.8078102452833033 rpy=0 0 0, axis 0 1 0, limit lower=-3.14159 upper=3.14159 effort=0.0 velocity=0.0
- added joint Link4_Link4ZeroLink0: type revolute, parent Link4, child Link4ZeroLink0, origin xyz=0.6042232109372674 0.6195297769938823 0 rpy=0 0 0, axis 0 1 0, limit lower=-3.14159 upper=3.14159 effort=0.0 velocity=0.0
- added joint Link4_Link5: type revolute, parent Link4, child Link5, origin xyz=0 1.2390595539877647 0 rpy=0 0 0, axis 0 1 0, limit lower=-3.14159 upper=3.14159 effort=0.0 velocity=0.0
- added joint Link5TwoLink0_Link5TwoLink1: type revolute, parent Link5TwoLink0, child Link5TwoLink1, origin xyz=0 0 1.1331223389185459 rpy=0 0 0, axis 0 1 0, limit lower=-3.14159 upper=3.14159 effort=0.0 velocity=0.0
- added joint Link5TwoLink1_Link5TwoLink2: type revolute, parent Link5TwoLink1, child Link5TwoLink2, origin xyz=0 0 1.1331223389185459 rpy=0 0 0, axis 0 1 0, limit lower=-3.14159 upper=3.14159 effort=0.0 velocity=0.0
- added joint Link5TwoLink2_Link5TwoLink3: type revolute, parent Link5TwoLink2, child Link5TwoLink3, origin xyz=0 0 1.1331223389185459 rpy=0 0 0, axis 0 1 0, limit lower=-3.14159 upper=3.14159 effort=0.0 velocity=0.0
- added joint Link5TwoLink3_Link5TwoLink4: type revolute, parent Link5TwoLink3, child Link5TwoLink4, origin xyz=0 0 1.1331223389185459 rpy=0 0 0, axis 0 1 0, limit lower=-3.14159 upper=3.14159 effort=0.0 velocity=0.0
- added joint Link5_Link5TwoLink0: type revolute, parent Link5, child Link5TwoLink0, origin xyz=0 0.5605140501371512 0.7914743482590229 rpy=0 0 0, axis 0 1 0, limit lower=-3.14159 upper=3.14159 effort=0.0 velocity=0.0
- joint Link0_Link1: origin xyz=0.13465097443592403 0 0.547413055316397 rpy=0 0 0 -> xyz=0 0.33266638169173035 0.8995515245166902 rpy=0 0 0

Commit message: Added readme.

File: body.urdf (robot description, URDF)
Before this commit: robot robot, 35 links, 34 joints
Links:
- removed link Link1TwoLink0
- removed link Link1TwoLink1
- removed link Link1TwoLink2
- removed link Link1TwoLink3
- removed link Link1TwoLink4
- removed link Link1ZeroLink0
- removed link Link2TwoLink0
- removed link Link2TwoLink1
- removed link Link2TwoLink2
- removed link Link2ZeroLink0
- removed link Link3OneLink0
- removed link Link3TwoLink0
- removed link Link3TwoLink1
- removed link Link3TwoLink2
- removed link Link3TwoLink3
- removed link Link3TwoLink4
- removed link Link3ZeroLink0
- removed link Link4OneLink0
- removed link Link4TwoLink0
- removed link Link4TwoLink1
- removed link Link4TwoLink2
- removed link Link4TwoLink3
- removed link Link4TwoLink4
- removed link Link4ZeroLink0
- removed link Link5TwoLink0
- removed link Link5TwoLink1
- removed link Link5TwoLink2
- removed link Link5TwoLink3
- removed link Link5TwoLink4
- added link Link6, mass 1; collision box size=0.291133517565908 1.5853115310517134 1.2335393436413413; visual box size=0.291133517565908 1.5853115310517134 1.2335393436413413
- added link Link7, mass 1; collision box size=1.5187752810576274 0.48314214776636355 1.2976490363209365; visual box size=1.5187752810576274 0.48314214776636355 1.2976490363209365
- link Link0: geometry collision box size=0.36875231222214033 1.2932231111382055 0.8000523993181177; visual box size=0.36875231222214033 1.2932231111382055 0.8000523993181177
- link Link1: geometry collision box size=1.780524806275726 0.6338014103448564 1.25379263878759; visual box size=1.780524806275726 0.6338014103448564 1.25379263878759
- link Link2: geometry collision box size=1.5363856724700766 0.6344002430494278 0.3067084692721084; visual box size=1.5363856724700766 0.6344002430494278 0.3067084692721084
- link Link3: geometry collision box size=0.9071918974946287 0.6067659323111304 0.26758196682411434; visual box size=0.9071918974946287 0.6067659323111304 0.26758196682411434
- link Link4: geometry collision box size=1.024168318867519 0.5565089356946695 1.1914352232948846; visual box size=1.024168318867519 0.5565089356946695 1.1914352232948846
- link Link5: geometry collision box size=1.1588925663621916 0.8844184217997275 1.6450923890315101; visual box size=1.1588925663621916 0.8844184217997275 1.6450923890315101
Joints:
- removed joint Link1TwoLink0_Link1TwoLink1
- removed joint Link1TwoLink1_Link1TwoLink2
- removed joint Link1TwoLink2_Link1TwoLink3
- removed joint Link1TwoLink3_Link1TwoLink4
- removed joint Link1_Link1TwoLink0
- removed joint Link1_Link1ZeroLink0
- removed joint Link2TwoLink0_Link2TwoLink1
- removed joint Link2TwoLink1_Link2TwoLink2
- removed joint Link2_Link2TwoLink0
- removed joint Link2_Link2ZeroLink0
- removed joint Link3TwoLink0_Link3TwoLink1
- removed joint Link3TwoLink1_Link3TwoLink2
- removed joint Link3TwoLink2_Link3TwoLink3
- removed joint Link3TwoLink3_Link3TwoLink4
- removed joint Link3_Link3OneLink0
- removed joint Link3_Link3TwoLink0
- removed joint Link3_Link3ZeroLink0
- removed joint Link4TwoLink0_Link4TwoLink1
- removed joint Link4TwoLink1_Link4TwoLink2
- removed joint Link4TwoLink2_Link4TwoLink3
- removed joint Link4TwoLink3_Link4TwoLink4
- removed joint Link4_Link4OneLink0
- removed joint Link4_Link4TwoLink0
- removed joint Link4_Link4ZeroLink0
- removed joint Link5TwoLink0_Link5TwoLink1
- removed joint Link5TwoLink1_Link5TwoLink2
- removed joint Link5TwoLink2_Link5TwoLink3
- removed joint Link5TwoLink3_Link5TwoLink4
- removed joint Link5_Link5TwoLink0
- added joint Link5_Link6: type revolute, parent Link5, child Link6, origin xyz=0 0.8844184217997275 0 rpy=0 0 0, axis 0 1 0, limit lower=-3.14159 upper=3.14159 effort=0.0 velocity=0.0
- added joint Link6_Link7: type revolute, parent Link6, child Link7, origin xyz=0 1.5853115310517134 0 rpy=0 0 0, axis 0 1 0, limit lower=-3.14159 upper=3.14159 effort=0.0 velocity=0.0
- joint Link0_Link1: origin xyz=0 0.33266638169173035 0.8995515245166902 rpy=0 0 0 -> xyz=0 0.6466115555691028 0.8225461945157551 rpy=0 0 0
- joint Link1_Link2: origin xyz=0 1.1339874684731799 0 rpy=0 0 0 -> xyz=0 0.6338014103448564 0 rpy=0 0 0
- joint Link2_Link3: origin xyz=0 1.4283480197268903 0 rpy=0 0 0 -> xyz=0 0.6344002430494278 0 rpy=0 0 0
- joint Link3_Link4: origin xyz=0 1.4578655587551734 0 rpy=0 0 0 -> xyz=0 0.6067659323111304 0 rpy=0 0 0
- joint Link4_Link5: origin xyz=0 1.2390595539877647 0 rpy=0 0 0 -> xyz=0 0.5565089356946695 0 rpy=0 0 0

Commit message: Checkpoint

File: body.urdf (robot description, URDF)
Before this commit: robot robot, 8 links, 7 joints
Links:
- removed link Link5
- removed link Link6
- removed link Link7
- link Link0: geometry collision box size=1.5257896326302387 1.5782735822799452 1.7742074208946892; visual box size=1.5257896326302387 1.5782735822799452 1.7742074208946892
- link Link1: geometry collision box size=1.683145725207021 0.7973269313857054 1.5150936824649357; visual box size=1.683145725207021 0.7973269313857054 1.5150936824649357
- link Link2: geometry collision box size=1.551977667392573 0.33525536279072676 0.29752474395061307; visual box size=1.551977667392573 0.33525536279072676 0.29752474395061307
- link Link3: geometry collision box size=1.4489517145571766 0.48363680955048505 1.0672299755897956; visual box size=1.4489517145571766 0.48363680955048505 1.0672299755897956
- link Link4: geometry collision box size=0.23320692054957776 0.7960509894622956 0.6257586957054899; visual box size=0.23320692054957776 0.7960509894622956 0.6257586957054899
Joints:
- removed joint Link4_Link5
- removed joint Link5_Link6
- removed joint Link6_Link7
- joint Link0_Link1: origin xyz=0 0.6466115555691028 0.8225461945157551 rpy=0 0 0 -> xyz=0 0.7891367911399726 0.8871037104473446 rpy=0 0 0
- joint Link1_Link2: origin xyz=0 0.6338014103448564 0 rpy=0 0 0 -> xyz=0 0.7973269313857054 0 rpy=0 0 0
- joint Link2_Link3: origin xyz=0 0.6344002430494278 0 rpy=0 0 0 -> xyz=0 0.33525536279072676 0 rpy=0 0 0
- joint Link3_Link4: origin xyz=0 0.6067659323111304 0 rpy=0 0 0 -> xyz=0 0.48363680955048505 0 rpy=0 0 0
